Commit message: Restructure repo: proper cell separation, launchers, current docs
- Rename fr_test_cell -> unchained_cell (package, module, launches, URDF;
  all references updated; both cells rebuilt & smoke-tested)
- CAD organized into cad/{pxrd,unchained}/ with meaningful names
  (check_v2.STL -> tabbed_plate_v2.STL etc.) + cad/README.md
- One-command launchers: run_pxrd.sh / run_unchained.sh with canonical
  validated args baked in (sim/load/retrieve/home/recover; sim/bridge/
  hw-scene/pick/home/stop)
- CLAUDE.md rewritten to reflect the actual current architecture (was the
  stale March plan); new docs/pxrd-cell.md + docs/unchained-cell.md with
  the validated constants and procedures; README.md quickstart

Co-Authored-By: Claude Fable 5 <noreply@anthropic.com>

File: ros2_ws/src/unchained_cell/urdf/dh_ag145_macro.xacro (robot description, xacro)
@@ -5,5 +5,5 @@
   with mesh paths repointed to our package and transmissions stripped.
   Usage:
-    <xacro:include filename="$(find fr_test_cell)/urdf/dh_ag145_macro.xacro"/>
+    <xacro:include filename="$(find unchained_cell)/urdf/dh_ag145_macro.xacro"/>
     <xacro:dh_ag145_gripper parent="wrist3_link" prefix="">
       <origin xyz="0 0 0" rpy="0 0 0"/>
@@ -27,10 +27,10 @@
       <visual>
         <geometry>
-          <mesh filename="package://fr_test_cell/meshes/dh_ag145/base_link.STL"/>
+          <mesh filename="package://unchained_cell/meshes/dh_ag145/base_link.STL"/>
         </geometry>
       </visual>
       <collision>
         <geometry>
-          <mesh filename="package://fr_test_cell/meshes/dh_ag145/base_link.STL"/>
+          <mesh filename="package://unchained_cell/meshes/dh_ag145/base_link.STL"/>
         </geometry>
       </collision>
@@ -59,8 +59,8 @@
     <link name="${prefix}gripper_finger1_knuckle_link">
       <visual>
-        <geometry><mesh filename="package://fr_test_cell/meshes/dh_ag145/crank_Link.STL"/></geometry>
-      </visual>
-      <collision>
-        <geometry><mesh filename="package://fr_test_cell/meshes/dh_ag145/crank_Link.STL"/></geometry>
+        <geometry><mesh filename="package://unchained_cell/meshes/dh_ag145/crank_Link.STL"/></geometry>
+      </visual>
+      <collision>
+        <geometry><mesh filename="package://unchained_cell/meshes/dh_ag145/crank_Link.STL"/></geometry>
       </collision>
       <inertial>
@@ -73,8 +73,8 @@
     <link name="${prefix}gripper_finger2_knuckle_link">
       <visual>
-        <geometry><mesh filename="package://fr_test_cell/meshes/dh_ag145/crank_Link.STL"/></geometry>
-      </visual>
-      <collision>
-        <geometry><mesh filename="package://fr_test_cell/meshes/dh_ag145/crank_Link.STL"/></geometry>
+        <geometry><mesh filename="package://unchained_cell/meshes/dh_ag145/crank_Link.STL"/></geometry>
+      </visual>
+      <collision>
+        <geometry><mesh filename="package://unchained_cell/meshes/dh_ag145/crank_Link.STL"/></geometry>
       </collision>
       <inertial>
@@ -103,8 +103,8 @@
     <link name="${prefix}gripper_finger1_finger_link">
       <visual>
-        <geometry><mesh filename="package://fr_test_cell/meshes/dh_ag145/rod_Link.STL"/></geometry>
-      </visual>
-      <collision>
-        <geometry><mesh filename="package://fr_test_cell/meshes/dh_ag145/rod_Link.STL"/></geometry>
+        <geometry><mesh filename="package://unchained_cell/meshes/dh_ag145/rod_Link.STL"/></geometry>
+      </visual>
+      <collision>
+        <geometry><mesh filename="package://unchained_cell/meshes/dh_ag145/rod_Link.STL"/></geometry>
       </collision>
       <inertial>
@@ -117,8 +117,8 @@
     <link name="${prefix}gripper_finger2_finger_link">
       <visual>
-        <geometry><mesh filename="package://fr_test_cell/meshes/dh_ag145/rod_Link.STL"/></geometry>
-      </visual>
-      <collision>
-        <geometry><mesh filename="package://fr_test_cell/meshes/dh_ag145/rod_Link.STL"/></geometry>
+        <geometry><mesh filename="package://unchained_cell/meshes/dh_ag145/rod_Link.STL"/></geometry>
+      </visual>
+      <collision>
+        <geometry><mesh filename="package://unchained_cell/meshes/dh_ag145/rod_Link.STL"/></geometry>
       </collision>
       <inertial>
@@ -147,8 +147,8 @@
     <link name="${prefix}gripper_finger1_inner_knuckle_link">
       <visual>
-        <geometry><mesh filename="package://fr_test_cell/meshes/dh_ag145/proximal_phalanx_Link.STL"/></geometry>
-      </visual>
-      <collision>
-        <geometry><mesh filename="package://fr_test_cell/meshes/dh_ag145/proximal_phalanx_Link.STL"/></geometry>
+        <geometry><mesh filename="package://unchained_cell/meshes/dh_ag145/proximal_phalanx_Link.STL"/></geometry>
+      </visual>
+      <collision>
+        <geometry><mesh filename="package://unchained_cell/meshes/dh_ag145/proximal_phalanx_Link.STL"/></geometry>
       </collision>
       <inertial>
@@ -161,8 +161,8 @@
     <link name="${prefix}gripper_finger2_inner_knuckle_link">
       <visual>
-        <geometry><mesh filename="package://fr_test_cell/meshes/dh_ag145/proximal_phalanx_Link.STL"/></geometry>
-      </visual>
-      <collision>
-        <geometry><mesh filename="package://fr_test_cell/meshes/dh_ag145/proximal_phalanx_Link.STL"/></geometry>
+        <geometry><mesh filename="package://unchained_cell/meshes/dh_ag145/proximal_phalanx_Link.STL"/></geometry>
+      </visual>
+      <collision>
+        <geometry><mesh filename="package://unchained_cell/meshes/dh_ag145/proximal_phalanx_Link.STL"/></geometry>
       </collision>
       <inertial>
@@ -191,8 +191,8 @@
     <link name="${prefix}gripper_finger1_finger_tip_link">
       <visual>
-        <geometry><mesh filename="package://fr_test_cell/meshes/dh_ag145/distal_phalanx_Link.STL"/></geometry>
-      </visual>
-      <collision>
-        <geometry><mesh filename="package://fr_test_cell/meshes/dh_ag145/distal_phalanx_Link.STL"/></geometry>
+        <geometry><mesh filename="package://unchained_cell/meshes/dh_ag145/distal_phalanx_Link.STL"/></geometry>
+      </visual>
+      <collision>
+        <geometry><mesh filename="package://unchained_cell/meshes/dh_ag145/distal_phalanx_Link.STL"/></geometry>
       </collision>
       <inertial>
@@ -205,8 +205,8 @@
     <link name="${prefix}gripper_finger2_finger_tip_link">
       <visual>
-        <geometry><mesh filename="package://fr_test_cell/meshes/dh_ag145/distal_phalanx_Link.STL"/></geometry>
-      </visual>
-      <collision>
-        <geometry><mesh filename="package://fr_test_cell/meshes/dh_ag145/distal_phalanx_Link.STL"/></geometry>
+        <geometry><mesh filename="package://unchained_cell/meshes/dh_ag145/distal_phalanx_Link.STL"/></geometry>
+      </visual>
+      <collision>
+        <geometry><mesh filename="package://unchained_cell/meshes/dh_ag145/distal_phalanx_Link.STL"/></geometry>
       </collision>
       <inertial>

File: ros2_ws/src/unchained_cell/urdf/unchained_cell.urdf.xacro (robot description, xacro)
@@ -9,6 +9,6 @@
   To add a test object, uncomment or copy the example block at the bottom.
   Usage:
-    xacro fr_test_cell.urdf.xacro robot_model:=fr16 control_mode:=gazebo
-    xacro fr_test_cell.urdf.xacro robot_model:=fr10 control_mode:=mock
+    xacro unchained_cell.urdf.xacro robot_model:=fr16 control_mode:=gazebo
+    xacro unchained_cell.urdf.xacro robot_model:=fr10 control_mode:=mock
 -->
 <robot xmlns:xacro="http://www.ros.org/wiki/xacro" name="fairino_v6_robot">
@@ -36,5 +36,5 @@
       <origin xyz="0 0 0" rpy="0 0 0"/>
       <geometry>
-        <mesh filename="package://fr_test_cell/meshes/pedestal_585mm.stl"
+        <mesh filename="package://unchained_cell/meshes/pedestal_585mm.stl"
               scale="0.001 0.001 0.001"/>
       </geometry>
@@ -46,5 +46,5 @@
       <origin xyz="0 0 0" rpy="0 0 0"/>
       <geometry>
-        <mesh filename="package://fr_test_cell/meshes/pedestal_585mm.stl"
+        <mesh filename="package://unchained_cell/meshes/pedestal_585mm.stl"
               scale="0.001 0.001 0.001"/>
       </geometry>
@@ -118,5 +118,5 @@
         <origin xyz="0 0 0" rpy="0 0 0"/>
         <geometry>
-          <mesh filename="package://fr_test_cell/meshes/unchained_junior_visual.stl"
+          <mesh filename="package://unchained_cell/meshes/unchained_junior_visual.stl"
                 scale="0.001 0.001 0.001"/>
         </geometry>
@@ -126,5 +126,5 @@
         <origin xyz="0 0 0" rpy="0 0 0"/>
         <geometry>
-          <mesh filename="package://fr_test_cell/meshes/unchained_junior_collision.stl"
+          <mesh filename="package://unchained_cell/meshes/unchained_junior_collision.stl"
                 scale="0.001 0.001 0.001"/>
         </geometry>

File: ros2_ws/src/unchained_cell/urdf/unchained_full.urdf.xacro (robot description, xacro)
@@ -52,5 +52,5 @@
       <origin xyz="0 0 0" rpy="0 0 0"/>
       <geometry>
-        <mesh filename="package://fr_test_cell/meshes/unchained_junior_visual.stl"
+        <mesh filename="package://unchained_cell/meshes/unchained_junior_visual.stl"
               scale="0.001 0.001 0.001"/>
       </geometry>
@@ -60,5 +60,5 @@
       <origin xyz="0 0 0" rpy="0 0 0"/>
       <geometry>
-        <mesh filename="package://fr_test_cell/meshes/unchained_junior_collision.stl"
+        <mesh filename="package://unchained_cell/meshes/unchained_junior_collision.stl"
               scale="0.001 0.001 0.001"/>
       </geometry>
@@ -236,5 +236,5 @@
       <origin xyz="0 0 0" rpy="0 0 0"/>
       <geometry>
-        <mesh filename="package://fr_test_cell/meshes/vention_pedestal_visual.stl"
+        <mesh filename="package://unchained_cell/meshes/vention_pedestal_visual.stl"
               scale="0.001 0.001 0.001"/>
       </geometry>
@@ -244,5 +244,5 @@
       <origin xyz="0 0 0" rpy="0 0 0"/>
       <geometry>
-        <mesh filename="package://fr_test_cell/meshes/vention_pedestal_collision.stl"
+        <mesh filename="package://unchained_cell/meshes/vention_pedestal_collision.stl"
               scale="0.001 0.001 0.001"/>
       </geometry>
@@ -264,5 +264,5 @@
     Plus an optional yaw to match real-world mounting orientation.
   -->
-  <xacro:include filename="$(find fr_test_cell)/urdf/fairino_armonly/fairino${robot_num}_v6_armonly.urdf"/>
+  <xacro:include filename="$(find unchained_cell)/urdf/fairino_armonly/fairino${robot_num}_v6_armonly.urdf"/>
   <joint name="robot_mount_joint" type="fixed">
     <parent link="pedestal"/>
@@ -328,5 +328,5 @@
   <!-- ============ AG-145 Gripper attached to wrist3_link ============ -->
   <xacro:if value="${'$(arg include_gripper)' == 'true'}">
-    <xacro:include filename="$(find fr_test_cell)/urdf/dh_ag145_macro.xacro"/>
+    <xacro:include filename="$(find unchained_cell)/urdf/dh_ag145_macro.xacro"/>
     <xacro:dh_ag145_gripper parent="wrist3_link" prefix="">
       <origin xyz="$(arg gripper_mount_x) $(arg gripper_mount_y) $(arg gripper_mount_z)"

File: ros2_ws/src/unchained_cell/urdf/unchained_only.urdf.xacro (robot description, xacro)
@@ -23,5 +23,5 @@
       <origin xyz="0 0 0" rpy="0 0 0"/>
       <geometry>
-        <mesh filename="package://fr_test_cell/meshes/unchained_junior_visual.stl"
+        <mesh filename="package://unchained_cell/meshes/unchained_junior_visual.stl"
               scale="0.001 0.001 0.001"/>
       </geometry>
@@ -33,5 +33,5 @@
       <origin xyz="0 0 0" rpy="0 0 0"/>
       <geometry>
-        <mesh filename="package://fr_test_cell/meshes/unchained_junior_collision.stl"
+        <mesh filename="package://unchained_cell/meshes/unchained_junior_collision.stl"
               scale="0.001 0.001 0.001"/>
       </geometry>
@@ -85,5 +85,5 @@
         <origin xyz="0 0 0" rpy="0 0 0"/>
         <geometry>
-          <mesh filename="package://fr_test_cell/meshes/vention_pedestal_visual.stl"
+          <mesh filename="package://unchained_cell/meshes/vention_pedestal_visual.stl"
                 scale="0.001 0.001 0.001"/>
         </geometry>
@@ -93,5 +93,5 @@
         <origin xyz="0 0 0" rpy="0 0 0"/>
         <geometry>
-          <mesh filename="package://fr_test_cell/meshes/vention_pedestal_collision.stl"
+          <mesh filename="package://unchained_cell/meshes/vention_pedestal_collision.stl"
                 scale="0.001 0.001 0.001"/>
         </geometry>
