Commit message: Unchained refit: new instrument scan, plate stand, tall rack types, tilt limits — fully sim-validated
Scene: new carved Unchained scan (9-10 rail restored into collision mesh after
decimation loss), synthetic obstacle box retired, hull SRDF whitelists removed
(honest gripper-vs-instrument), plate_stand w/ stand_pos1..6 on the AMR table
(baked defaults world -0.3/-1.7 h0.75), wp_sd/8ml/20ml rack meshes.

Motion: --plate-type with per-height grasp math + mesh ACOs; tilt hard limit
±2° default-on for all carried phases (open vials); grasp-relative hover
(fixes 9-10 approach + vortex_pos2 graze — one bug, three symptoms); OMPL
longest_valid_segment_fraction=0.002 (thin-sheet visibility); purge ordering
fix BOTH cells (detach-then-remove; MoveIt re-inserts detached ACOs into world).

Validated via parallel agent sims (strict collision, tilt on): all 6 stand
positions pickable w/ 5 neighbors; vortex pos1+2 pass (sim==reality);
deck_9_10_pos1 pickable WITH the rail (30.9mm gap vs 7-10mm fingertip).
Playbook §9 records the transferable lessons.

Co-Authored-By: Claude Fable 5 <noreply@anthropic.com>

File: ros2_ws/src/unchained_cell/urdf/unchained_full.urdf.xacro (robot description, xacro)
@@ -76,5 +76,8 @@
   </joint>
   <!-- ================ Deck markers (CAD frame) ================ -->
-  <xacro:macro name="deck_marker" params="name x y z">
+  <!-- Generic Y-up marker. Default parent is the Unchained (CAD frame);
+       pass parent:=plate_stand for the stand pockets. Both parents carry a
+       Y-up frame, so rpy=0 keeps every marker Y-up. -->
+  <xacro:macro name="deck_marker" params="name x y z parent:=unchained_junior">
     <link name="${name}">
       <visual>
@@ -85,5 +88,5 @@
     </link>
     <joint name="${name}_joint" type="fixed">
-      <parent link="unchained_junior"/>
+      <parent link="${parent}"/>
       <child link="${name}"/>
       <origin xyz="${x} ${y} ${z}" rpy="0 0 0"/>
@@ -97,38 +100,11 @@
   <xacro:deck_marker name="deck_vortex_pos3"    x="0.19001"  y="0.26004" z="0.62009"/>
   <xacro:deck_marker name="deck_vacuum_filtration" x="0.31345" y="0.26956" z="0.69374"/>
-  <!-- ============ Fixed obstacle next to deck_9_10_pos1 ============
-       A physical cuboid present on the real machine beside deck 9-10 pos 1.
-       Offset + size were measured in SolidWorks (CAD frame) relative to the
-       deck 1 CENTER. The deck marker frame shares the CAD axis orientation
-       (deck markers are rpy=0 children of unchained_junior, which carries the
-       CAD Y-up frame), so SolidWorks X/Y/Z map in directly — no axis swap;
-       the CAD->world Z-up conversion is handled by unchained_junior_joint.
-       SolidWorks center offset from deck1: x=-90, y=11.63, z=22.88 mm
-       Measured SolidWorks dims (x,y,z): 28.4 x 65 x 120 mm.
-       Box PADDED over the measured size for clearance (keep it big so the arm
-       reliably avoids the real obstacle): X 28.4->40, Y 65->100, Z 120->160.
-       Centered on the measured artifact center. NOTE: at this size the box
-       intrudes into the corridor the arm uses for deck_vortex_pos1 — handled
-       by raising that approach, not by shrinking the box.
-       Box origin = link frame = artifact center (offset is to the center). -->
-  <link name="obstacle_deck1">
-    <visual>
-      <origin xyz="0 0 0" rpy="0 0 0"/>
-      <geometry><box size="0.040 0.100 0.160"/></geometry>
-      <material name="obstacle_deck1_color"><color rgba="0.85 0.1 0.1 0.55"/></material>
-    </visual>
-    <collision>
-      <origin xyz="0 0 0" rpy="0 0 0"/>
-      <geometry><box size="0.040 0.100 0.160"/></geometry>
-    </collision>
-  </link>
-  <joint name="obstacle_deck1_joint" type="fixed">
-    <parent link="deck_9_10_pos1"/>
-    <child link="obstacle_deck1"/>
-    <origin xyz="-0.090 0.01163 0.02288" rpy="0 0 0"/>
-  </joint>
+  <!-- ============ Fixed obstacle next to deck_9_10_pos1 (REMOVED) ============
+       The synthetic obstacle_deck1 box was deleted: the real obstruction is
+       now part of the instrument collision mesh (new scan of the Unchained). -->
   <!-- ================ Lab table (loading station) ================
-       A 30×30×70 cm box next to the pedestal. The plate gets staged here
-       on the way out of (or into) the Unchained device.
+       An AMR-like table box next to the pedestal (default 60×60×75 cm; the
+       position defaults are a starting point for manual tuning). The plate
+       gets staged here on the way out of (or into) the Unchained device.
        Table position is in WORLD frame (Z-up). The `table_top` frame is a
        child of `table` with rpy="1.5708 0 0" so its local +Y axis points
@@ -137,10 +113,20 @@
        Tunable via include_table arg (default true) and the table_*_xyz args. -->
   <xacro:arg name="include_table" default="true"/>
-  <xacro:arg name="table_x" default="0.7"/>
-  <xacro:arg name="table_y" default="-1.3"/>
+  <xacro:arg name="table_x" default="-0.3"/>
+  <xacro:arg name="table_y" default="-1.7"/>
   <xacro:arg name="table_z" default="0.0"/>
-  <xacro:arg name="table_w" default="0.30"/>     <!-- width  (X) -->
-  <xacro:arg name="table_d" default="0.30"/>     <!-- depth  (Y) -->
-  <xacro:arg name="table_h" default="0.70"/>     <!-- height (Z) -->
+  <xacro:arg name="table_w" default="0.6"/>      <!-- width  (X) -->
+  <xacro:arg name="table_d" default="0.6"/>      <!-- depth  (Y) -->
+  <xacro:arg name="table_h" default="0.75"/>     <!-- height (Z) -->
+  <!-- Plate stand placement on the table top (table_top frame is Y-up:
+       local +Y = world up, X/Z span the table surface). -->
+  <xacro:arg name="stand_x" default="0.0"/>
+  <xacro:arg name="stand_y_up" default="0.0"/>
+  <xacro:arg name="stand_z" default="0.0"/>
+  <xacro:arg name="stand_yaw_deg" default="0"/>
+  <!-- Static wp_sd.stl plates at the stand markers, for layout eyeballing. -->
+  <xacro:arg name="include_stand_plates" default="false"/>
+  <xacro:property name="stand_yaw_deg_prop" value="$(arg stand_yaw_deg)"/>
+  <xacro:property name="stand_yaw_rad" value="${float(stand_yaw_deg_prop) * pi / 180.0}"/>
   <xacro:if value="${'$(arg include_table)' == 'true'}">
     <xacro:property name="tw" value="$(arg table_w)"/>
@@ -182,4 +168,82 @@
       <origin xyz="0 0 ${th}" rpy="1.5708 0 0"/>
     </joint>
+    <!-- ================ Plate stand on the table ================
+         Mesh native frame: origin at bottom center, Y-up, bbox 300×15.5×300 mm
+         — so at zero offsets it sits centered on the table top.
+         Parent table_top is Y-up (local +Y = world up), so:
+           - stand_y_up raises the stand off the table surface
+           - the yaw about the VERTICAL axis goes in the PITCH slot of rpy
+             (pitch = rotation about parent Y = true vertical here). -->
+    <link name="plate_stand">
+      <visual>
+        <origin xyz="0 0 0" rpy="0 0 0"/>
+        <geometry>
+          <mesh filename="package://unchained_cell/meshes/plate_stand.stl"
+                scale="0.001 0.001 0.001"/>
+        </geometry>
+        <material name="stand_grey"><color rgba="0.45 0.45 0.5 1.0"/></material>
+      </visual>
+      <collision>
+        <origin xyz="0 0 0" rpy="0 0 0"/>
+        <geometry>
+          <mesh filename="package://unchained_cell/meshes/plate_stand.stl"
+                scale="0.001 0.001 0.001"/>
+        </geometry>
+      </collision>
+      <inertial>
+        <mass value="2.0"/>
+        <inertia ixx="0.02" ixy="0" ixz="0" iyy="0.02" iyz="0" izz="0.02"/>
+      </inertial>
+    </link>
+    <joint name="plate_stand_joint" type="fixed">
+      <parent link="table_top"/>
+      <child link="plate_stand"/>
+      <origin xyz="$(arg stand_x) $(arg stand_y_up) $(arg stand_z)"
+              rpy="0 ${stand_yaw_rad} 0"/>
+    </joint>
+    <!-- Stand deck markers: 2×3 grid of pocket floors, Y-up like all deck
+         markers (rpy=0 relative to the stand, which is already Y-up).
+         y=0.0075 = pocket floor height above the stand bottom. -->
+    <xacro:deck_marker name="stand_pos1" parent="plate_stand" x="-0.070" y="0.0075" z="0.100"/>
+    <xacro:deck_marker name="stand_pos2" parent="plate_stand" x="-0.070" y="0.0075" z="0.000"/>
+    <xacro:deck_marker name="stand_pos3" parent="plate_stand" x="-0.070" y="0.0075" z="-0.100"/>
+    <xacro:deck_marker name="stand_pos4" parent="plate_stand" x="0.070" y="0.0075" z="0.100"/>
+    <xacro:deck_marker name="stand_pos5" parent="plate_stand" x="0.070" y="0.0075" z="0.000"/>
+    <xacro:deck_marker name="stand_pos6" parent="plate_stand" x="0.070" y="0.0075" z="-0.100"/>
+    <!-- Optional STATIC well-plate meshes at each stand marker, for
+         eyeballing the layout only. Runtime picks manage plates dynamically
+         (pick_place.py CollisionObjects), so this defaults OFF. -->
+    <xacro:if value="${'$(arg include_stand_plates)' == 'true'}">
+      <xacro:macro name="stand_plate_vis" params="marker">
+        <link name="${marker}_plate">
+          <visual>
+            <origin xyz="0 0 0" rpy="0 0 0"/>
+            <geometry>
+              <mesh filename="package://unchained_cell/meshes/wp_sd.stl"
+                    scale="0.001 0.001 0.001"/>
+            </geometry>
+            <material name="${marker}_plate_color"><color rgba="0.92 0.92 0.95 1.0"/></material>
+          </visual>
+          <collision>
+            <origin xyz="0 0 0" rpy="0 0 0"/>
+            <geometry>
+              <mesh filename="package://unchained_cell/meshes/wp_sd.stl"
+                    scale="0.001 0.001 0.001"/>
+            </geometry>
+          </collision>
+        </link>
+        <joint name="${marker}_plate_joint" type="fixed">
+          <parent link="${marker}"/>
+          <child link="${marker}_plate"/>
+          <origin xyz="0 0 0" rpy="0 0 0"/>
+        </joint>
+      </xacro:macro>
+      <xacro:stand_plate_vis marker="stand_pos1"/>
+      <xacro:stand_plate_vis marker="stand_pos2"/>
+      <xacro:stand_plate_vis marker="stand_pos3"/>
+      <xacro:stand_plate_vis marker="stand_pos4"/>
+      <xacro:stand_plate_vis marker="stand_pos5"/>
+      <xacro:stand_plate_vis marker="stand_pos6"/>
+    </xacro:if>
   </xacro:if>
   <!-- ================ Well-plate model ================

Commit message: Real table assembly replaces box stand-in — 20ml validated from all 8 pockets
- cad/unchained/table_asm.STL -> meshes/table_visual.stl + table_collision.stl
  (rotated to match prior layout: 400mm along X, 550mm along Y; origin at
  floor under table center; casters on the floor).
- Tabletop plane measured at 776.2mm (was 750 box): table_top frame moved,
  holder + stand_pos1..8 markers follow automatically.
- Perimeter bolt heads (+3.6mm, ~22mm in from edges) are in collision but
  clear of the centered holder footprint.
- Re-validated: 20ml load from ALL 8 pockets -> vortex pos1, strict
  collision checking, 8/8 PASS, zero retries.

Co-Authored-By: Claude Fable 5 <noreply@anthropic.com>

File: ros2_ws/src/unchained_cell/urdf/unchained_full.urdf.xacro (robot description, xacro)
@@ -133,16 +133,27 @@
   <xacro:property name="stand_yaw_rad" value="${float(stand_yaw_deg_prop) * pi / 180.0}"/>
   <xacro:if value="${'$(arg include_table)' == 'true'}">
-    <xacro:property name="tw" value="$(arg table_w)"/>
-    <xacro:property name="td" value="$(arg table_d)"/>
-    <xacro:property name="th" value="$(arg table_h)"/>
+    <!-- Real table assembly (cad/unchained/table_asm.STL, 2026-10-02):
+         550 x 400 frame on casters, converted so the link origin is at the
+         FLOOR under the table center, long (550) side along world Y (same
+         orientation as the old 400x550 box). TABLETOP PLANE = +0.7762m
+         (casters 20.2mm + frame; perimeter bolt heads rise to 779.8mm but
+         sit ~22mm in from the edges, OUTSIDE the centered holder footprint).
+         table_w/d/h launch args no longer shape the geometry. -->
+    <xacro:property name="table_top_z" value="0.7762"/>
     <link name="table">
       <visual>
-        <origin xyz="0 0 ${th/2}" rpy="0 0 0"/>
-        <geometry><box size="${tw} ${td} ${th}"/></geometry>
-        <material name="wood"><color rgba="0.55 0.35 0.18 1.0"/></material>
+        <origin xyz="0 0 0" rpy="${pi/2} 0 0"/>
+        <geometry>
+          <mesh filename="package://unchained_cell/meshes/table_visual.stl"
+                scale="0.001 0.001 0.001"/>
+        </geometry>
+        <material name="table_alu"><color rgba="0.62 0.62 0.66 1.0"/></material>
       </visual>
       <collision>
-        <origin xyz="0 0 ${th/2}" rpy="0 0 0"/>
-        <geometry><box size="${tw} ${td} ${th}"/></geometry>
+        <origin xyz="0 0 0" rpy="${pi/2} 0 0"/>
+        <geometry>
+          <mesh filename="package://unchained_cell/meshes/table_collision.stl"
+                scale="0.001 0.001 0.001"/>
+        </geometry>
       </collision>
       <inertial>
@@ -167,7 +178,7 @@
       <parent link="table"/>
       <child link="table_top"/>
-      <!-- xyz: at top-center of table. rpy="π/2 0 0" rotates so table_top
-           local +Y points along world +Z (up). -->
-      <origin xyz="0 0 ${th}" rpy="1.5708 0 0"/>
+      <!-- xyz: at the TABLETOP PLANE of the mesh. rpy="π/2 0 0" rotates so
+           table_top local +Y points along world +Z (up). -->
+      <origin xyz="0 0 ${table_top_z}" rpy="1.5708 0 0"/>
     </joint>
     <!-- ================ Plate stand on the table ================

Commit message: Pedestal as-built correction: +5mm from machine, 2deg CW — trio follows
User-observed after bolting: pedestal joint origin +5mm local Z and
-2deg about vertical. The arm rides the pedestal, so its WORLD yaw is
now -137: GRASP_YAW_COMP_DEG 137 and HOME j1 +137deg follow (the
pedestal-relative robot_mount_yaw_deg stays -135 — physically unchanged).
Sim-validated: 20ml all-pocket round trips + 8ml/96 spots; the single
pos3-load failure reproduced 0/3 on a clean sim (seed fluke, duplicate-
scene noise in the matrix run).

Co-Authored-By: Claude Fable 5 <noreply@anthropic.com>

File: ros2_ws/src/unchained_cell/urdf/unchained_full.urdf.xacro (robot description, xacro)
@@ -345,5 +345,10 @@
     <parent link="unchained_junior"/>
     <child link="pedestal"/>
-    <origin xyz="0.400 0.31533 1.13827" rpy="0 0 0"/>
+    <!-- AS-BUILT pedestal calibration (2026-10-28, user-observed after
+       bolting): +5mm away from the machine (local +Z) and 2deg clockwise
+       from above (-2deg about vertical = pitch slot in this Y-up frame).
+       NOTE: this also yaws the ARM riding the pedestal -> the coupled trio
+       (GRASP_YAW_COMP_DEG=137, HOME j1=+137deg) moved with it. -->
+    <origin xyz="0.400 0.31533 1.14327" rpy="0 ${-2*pi/180} 0"/>
   </joint>
   <!-- ================ FR16 robot (arm chain only, no world link) ================ -->
