Commit message: Unchained refit round 2: un-mirror gripper model, calibrate aperture, auto grip width, 8-pocket holder — 20ml validated from all 8 pockets
- dh_ag145_macro.xacro (both cells): gripper model rendered joint 0.0 as
  CLOSED, mirrored vs the hardware-verified convention (0=SDK 100%=open).
  Axis-flip + baked origin rotations; joint values/limits unchanged so all
  hardware-proven code paths are untouched.
- mimic_repeater node: publishes the 7 mimic gripper joints so rviz renders
  the true gripper (display lied for the whole project until now).
- pick_place: FK-calibrated cubic aperture map (full open = 148.7mm true pad
  gap); AUTO grip width per source deck (long side 128.5mm at stand pockets,
  short side 86.1mm at vortex nest); per-rack grip_center heights; per-deck
  rest float (stand/table seat flush 0.5mm, nests keep measured 5mm).
- New wellplate_holder (350x500, 8 pockets 2x4, corner fins) + accurate
  8ml/20ml rack meshes; markers stand_pos1..8 on pocket floors.
- Table (AMR stand-in) now 400x550x750 at (-0.4,-1.7): fixes carry-home
  planning failures from pockets 7/8; 20ml load validated from ALL 8
  pockets to vortex pos1 under full strict collision checking.
- Stock AG-145 fingers confirmed sufficient — no extensions needed (old
  conclusion was an artifact of the mirrored model + wrong grip width).
- CAD sources moved to cad/unchained/; docs/unchained-refit-handoff.md
  captures full session state and open items.

Co-Authored-By: Claude Fable 5 <noreply@anthropic.com>

File: ros2_ws/src/pxrd_cell/urdf/dh_ag145_macro.xacro (robot description, xacro)
@@ -42,9 +42,17 @@
       </inertial>
     </link>
+    <!-- SIGN CONVENTION FIX (measured 2026-09): the original model rendered
+         joint 0.0 as jaws CLOSED (18mm tip separation) and -0.65 as OPEN
+         (161mm), i.e. mirrored vs the real AG-145 + fr_bridge mapping
+         (0.0 = SDK 100% = open, -0.65 = SDK 0% = closed, hardware-verified).
+         Fix: every gripper joint has its axis flipped and a constant
+         0.65*multiplier rotation baked into its origin, so joint value v now
+         renders what the old model rendered at (-0.65 - v). Joint VALUES and
+         limits are unchanged -> all software & bridge conventions intact. -->
     <joint name="${prefix}gripper_finger1_joint" type="revolute">
       <parent link="${prefix}gripper_base_link"/>
       <child link="${prefix}gripper_finger1_knuckle_link"/>
-      <axis xyz="0 -1 0"/>
-      <origin rpy="0.0 0.0 ${pi}" xyz="-0.016 0 0.10586"/>
+      <axis xyz="0 1 0"/>
+      <origin rpy="0 0.650000 ${pi}" xyz="-0.016 0 0.10586"/>
       <limit lower="-0.65" upper="0.0" velocity="100.0" effort="1000"/>
     </joint>
@@ -52,6 +60,6 @@
       <parent link="${prefix}gripper_base_link"/>
       <child link="${prefix}gripper_finger2_knuckle_link"/>
-      <axis xyz="0 -1 0"/>
-      <origin rpy="0.0 0.0 0.0" xyz="0.016 0 0.10586"/>
+      <axis xyz="0 1 0"/>
+      <origin rpy="0 0.650000 0.0" xyz="0.016 0 0.10586"/>
       <limit lower="-3.14" upper="3.14" velocity="100.0" effort="1000"/>
       <mimic joint="${prefix}gripper_finger1_joint"/>
@@ -88,6 +96,6 @@
       <parent link="${prefix}gripper_finger1_knuckle_link"/>
       <child link="${prefix}gripper_finger1_finger_link"/>
-      <axis xyz="0 -1 0"/>
-      <origin xyz="0.036999 0 -0.00019698" rpy="0 0 0"/>
+      <axis xyz="0 1 0"/>
+      <origin xyz="0.036999 0 -0.00019698" rpy="0 0.325000 0"/>
       <limit lower="-3.14" upper="3.14" velocity="100.0" effort="105"/>
       <mimic joint="${prefix}gripper_finger1_joint" multiplier="0.5" offset="0"/>
@@ -96,6 +104,6 @@
       <parent link="${prefix}gripper_finger2_knuckle_link"/>
       <child link="${prefix}gripper_finger2_finger_link"/>
-      <axis xyz="0 -1 0"/>
-      <origin xyz="0.036999 0 -0.00019698" rpy="0 0 0"/>
+      <axis xyz="0 1 0"/>
+      <origin xyz="0.036999 0 -0.00019698" rpy="0 0.325000 0"/>
       <limit lower="-3.14" upper="3.14" velocity="100.0" effort="105"/>
       <mimic joint="${prefix}gripper_finger1_joint" multiplier="0.5" offset="0"/>
@@ -132,6 +140,6 @@
       <parent link="${prefix}gripper_base_link"/>
       <child link="${prefix}gripper_finger1_inner_knuckle_link"/>
-      <axis xyz="0 -1 0"/>
-      <origin rpy="0.0 0.0 ${pi}" xyz="-0.016 0 0.10586"/>
+      <axis xyz="0 1 0"/>
+      <origin rpy="0 0.968500 ${pi}" xyz="-0.016 0 0.10586"/>
       <limit lower="-3.14" upper="3.14" velocity="100.0" effort="105"/>
       <mimic joint="${prefix}gripper_finger1_joint" multiplier="1.49" offset="0"/>
@@ -140,6 +148,6 @@
       <parent link="${prefix}gripper_base_link"/>
       <child link="${prefix}gripper_finger2_inner_knuckle_link"/>
-      <axis xyz="0 -1 0"/>
-      <origin rpy="0.0 0.0 0.0" xyz="0.016 0 0.10586"/>
+      <axis xyz="0 1 0"/>
+      <origin rpy="0 0.968500 0.0" xyz="0.016 0 0.10586"/>
       <limit lower="-3.14" upper="3.14" velocity="100.0" effort="105"/>
       <mimic joint="${prefix}gripper_finger1_joint" multiplier="1.49" offset="0"/>
@@ -176,6 +184,6 @@
       <parent link="${prefix}gripper_finger1_inner_knuckle_link"/>
       <child link="${prefix}gripper_finger1_finger_tip_link"/>
-      <axis xyz="0 1 0"/>
-      <origin xyz="-0.0081054 0 0.086119" rpy="0.0 0.0 0.0"/>
+      <axis xyz="0 -1 0"/>
+      <origin xyz="-0.0081054 0 0.086119" rpy="0 -0.968500 0.0"/>
       <limit lower="-3.14" upper="3.14" velocity="100.0" effort="0.1"/>
       <mimic joint="${prefix}gripper_finger1_joint" multiplier="1.49"/>
@@ -184,6 +192,6 @@
       <parent link="${prefix}gripper_finger2_inner_knuckle_link"/>
       <child link="${prefix}gripper_finger2_finger_tip_link"/>
-      <axis xyz="0 1 0"/>
-      <origin rpy="0.0 0.0 0.0" xyz="-0.0081054 0 0.086119"/>
+      <axis xyz="0 -1 0"/>
+      <origin rpy="0 -0.968500 0.0" xyz="-0.0081054 0 0.086119"/>
       <limit lower="-3.14" upper="3.14" velocity="100.0" effort="0.1"/>
       <mimic joint="${prefix}gripper_finger1_joint" multiplier="1.49"/>

File: ros2_ws/src/unchained_cell/urdf/unchained_full.urdf.xacro (robot description, xacro)
@@ -79,5 +79,5 @@
        pass parent:=plate_stand for the stand pockets. Both parents carry a
        Y-up frame, so rpy=0 keeps every marker Y-up. -->
-  <xacro:macro name="deck_marker" params="name x y z parent:=unchained_junior">
+  <xacro:macro name="deck_marker" params="name x y z parent:=unchained_junior yaw:=0">
     <link name="${name}">
       <visual>
@@ -90,5 +90,6 @@
       <parent link="${parent}"/>
       <child link="${name}"/>
-      <origin xyz="${x} ${y} ${z}" rpy="0 0 0"/>
+      <!-- yaw about the VERTICAL axis = pitch slot (parent frames are Y-up) -->
+      <origin xyz="${x} ${y} ${z}" rpy="0 ${yaw} 0"/>
     </joint>
   </xacro:macro>
@@ -125,5 +126,7 @@
   <xacro:arg name="stand_z" default="0.0"/>
   <xacro:arg name="stand_yaw_deg" default="0"/>
-  <!-- Static wp_sd.stl plates at the stand markers, for layout eyeballing. -->
+  <!-- Static well-plate meshes at the stand markers, for layout eyeballing.
+       stand_plate_mesh selects the rack type shown: wp_8ml / wp_20ml / wp_sd. -->
+  <xacro:arg name="stand_plate_mesh" default="wp_8ml"/>
   <xacro:arg name="include_stand_plates" default="false"/>
   <xacro:property name="stand_yaw_deg_prop" value="$(arg stand_yaw_deg)"/>
@@ -179,5 +182,5 @@
         <origin xyz="0 0 0" rpy="0 0 0"/>
         <geometry>
-          <mesh filename="package://unchained_cell/meshes/plate_stand.stl"
+          <mesh filename="package://unchained_cell/meshes/wellplate_holder.stl"
                 scale="0.001 0.001 0.001"/>
         </geometry>
@@ -187,5 +190,5 @@
         <origin xyz="0 0 0" rpy="0 0 0"/>
         <geometry>
-          <mesh filename="package://unchained_cell/meshes/plate_stand.stl"
+          <mesh filename="package://unchained_cell/meshes/wellplate_holder.stl"
                 scale="0.001 0.001 0.001"/>
         </geometry>
@@ -204,11 +207,22 @@
     <!-- Stand deck markers: 2×3 grid of pocket floors, Y-up like all deck
          markers (rpy=0 relative to the stand, which is already Y-up).
-         y=0.0075 = pocket floor height above the stand bottom. -->
-    <xacro:deck_marker name="stand_pos1" parent="plate_stand" x="-0.070" y="0.0075" z="0.100"/>
-    <xacro:deck_marker name="stand_pos2" parent="plate_stand" x="-0.070" y="0.0075" z="0.000"/>
-    <xacro:deck_marker name="stand_pos3" parent="plate_stand" x="-0.070" y="0.0075" z="-0.100"/>
-    <xacro:deck_marker name="stand_pos4" parent="plate_stand" x="0.070" y="0.0075" z="0.100"/>
-    <xacro:deck_marker name="stand_pos5" parent="plate_stand" x="0.070" y="0.0075" z="0.000"/>
-    <xacro:deck_marker name="stand_pos6" parent="plate_stand" x="0.070" y="0.0075" z="-0.100"/>
+         y=0.0155 = GUIDE-RAIL TOP: plates rest ON the rails (support ledges);
+         a floor-resting plate would intersect the rails where its long side
+         overhangs the 100mm pocket span (found via honest carried-plate
+         collision checking, 2026-09-23). -->
+    <!-- wellplate_holder (2026-09-24): 350x500x12.5mm plate, 8 recessed
+         pockets (2 cols x 4 rows), pocket 128.0 x 86.0mm, floor at y=7.5
+         (5mm deep). Plates SEAT ON THE POCKET FLOOR -> marker y=0.0075.
+         Pocket centers measured from the mesh: X=+-87.5, Z=+-62.5/+-187.5.
+         pos1-4 = col X=-0.0875 (rows Z +0.1875..-0.1875),
+         pos5-8 = col X=+0.0875 (same row order). -->
+    <xacro:deck_marker name="stand_pos1" parent="plate_stand" x="-0.0875" y="0.0075" z="0.1875" yaw="${pi/2}"/>
+    <xacro:deck_marker name="stand_pos2" parent="plate_stand" x="-0.0875" y="0.0075" z="0.0625" yaw="${pi/2}"/>
+    <xacro:deck_marker name="stand_pos3" parent="plate_stand" x="-0.0875" y="0.0075" z="-0.0625" yaw="${pi/2}"/>
+    <xacro:deck_marker name="stand_pos4" parent="plate_stand" x="-0.0875" y="0.0075" z="-0.1875" yaw="${pi/2}"/>
+    <xacro:deck_marker name="stand_pos5" parent="plate_stand" x="0.0875" y="0.0075" z="0.1875" yaw="${pi/2}"/>
+    <xacro:deck_marker name="stand_pos6" parent="plate_stand" x="0.0875" y="0.0075" z="0.0625" yaw="${pi/2}"/>
+    <xacro:deck_marker name="stand_pos7" parent="plate_stand" x="0.0875" y="0.0075" z="-0.0625" yaw="${pi/2}"/>
+    <xacro:deck_marker name="stand_pos8" parent="plate_stand" x="0.0875" y="0.0075" z="-0.1875" yaw="${pi/2}"/>
     <!-- Optional STATIC well-plate meshes at each stand marker, for
          eyeballing the layout only. Runtime picks manage plates dynamically
@@ -220,5 +234,5 @@
             <origin xyz="0 0 0" rpy="0 0 0"/>
             <geometry>
-              <mesh filename="package://unchained_cell/meshes/wp_sd.stl"
+              <mesh filename="package://unchained_cell/meshes/$(arg stand_plate_mesh).stl"
                     scale="0.001 0.001 0.001"/>
             </geometry>
@@ -228,5 +242,5 @@
             <origin xyz="0 0 0" rpy="0 0 0"/>
             <geometry>
-              <mesh filename="package://unchained_cell/meshes/wp_sd.stl"
+              <mesh filename="package://unchained_cell/meshes/$(arg stand_plate_mesh).stl"
                     scale="0.001 0.001 0.001"/>
             </geometry>
@@ -245,4 +259,6 @@
       <xacro:stand_plate_vis marker="stand_pos5"/>
       <xacro:stand_plate_vis marker="stand_pos6"/>
+      <xacro:stand_plate_vis marker="stand_pos7"/>
+      <xacro:stand_plate_vis marker="stand_pos8"/>
     </xacro:if>
   </xacro:if>
