Commit message: PXRD: DH AG-95 gripper support — sim-qualified drop-in alternative to the AG-145
New dh_ag95_macro.xacro wraps the vendored fairino-moveit2 AG-95 model
(four-bar fingers, all mimicking one actuated joint) with AG-145-compatible
link/joint names, so the SRDF masks, touch_links and the gripper controller
work unchanged. grasp_link_offset 0.114 keeps the pad center exactly
PAD_OFFSET_FROM_TCP (0.069) ahead of the TCP — no aiming constants change.

Selection: launch gripper:=ag145|ag95 + pick_place --gripper (GRIPPERS dict:
ag145 0..-0.65 over 145mm; ag95 0..+0.93 over 95.2mm, FK-measured).

Why the AG-95 fits this cell well (FK envelope analysis): NOTHING extends
beyond its pads toward the workspace — the ~37mm below-pad fingertip that
forced the v3 overhang margins on the AG-145 simply does not exist, so all
fingertip clearances gain margin.

Qualified in sim (v3 plate, canonical layout): full round trip green both
directions, 0 retries, carry level at 9.32 deg; the gripper swap correctly
flips the layout fingerprint, so the taught carry was re-validated with
the DENSE live collision check against the AG-95 geometry and passed.

Also: SRDF gains the AG-95 adjacency/four-bar-loop pairs (unknown-link
entries are ignored under the AG-145), gripper_body_link in touch links,
AG-95 meshes vendored into pxrd_cell/meshes/dh_ag95/.

Co-Authored-By: Claude Fable 5 <noreply@anthropic.com>

File: ros2_ws/src/pxrd_cell/urdf/pxrd_full.urdf.xacro (robot description, xacro)
@@ -380,11 +380,28 @@
     </gazebo>
   </xacro:if>
-  <!-- ============ AG-145 Gripper attached to wrist3_link ============ -->
+  <!-- ============ Gripper attached to wrist3_link ============
+       gripper:=ag145 (default) | ag95. Both macros expose the SAME link and
+       joint names (gripper_finger1_joint actuated, gripper_grasp_link TCP,
+       finger/knuckle/tip link names), so controllers, SRDF masks and
+       touch_links work for either. Joint conventions differ:
+         ag145: 0.0 = open (145 mm), -0.65 = closed
+         ag95 : 0.0 = open (95.2 mm), +0.93 = closed
+       pick_place maps grip widths per gripper via its - -gripper flag. -->
+  <xacro:arg name="gripper" default="ag145"/>
   <xacro:if value="${'$(arg include_gripper)' == 'true'}">
-    <xacro:include filename="$(find pxrd_cell)/urdf/dh_ag145_macro.xacro"/>
-    <xacro:dh_ag145_gripper parent="wrist3_link" prefix="">
-      <origin xyz="$(arg gripper_mount_x) $(arg gripper_mount_y) $(arg gripper_mount_z)"
-              rpy="$(arg gripper_mount_roll) $(arg gripper_mount_pitch) $(arg gripper_mount_yaw)"/>
-    </xacro:dh_ag145_gripper>
+    <xacro:if value="${'$(arg gripper)' == 'ag145'}">
+      <xacro:include filename="$(find pxrd_cell)/urdf/dh_ag145_macro.xacro"/>
+      <xacro:dh_ag145_gripper parent="wrist3_link" prefix="">
+        <origin xyz="$(arg gripper_mount_x) $(arg gripper_mount_y) $(arg gripper_mount_z)"
+                rpy="$(arg gripper_mount_roll) $(arg gripper_mount_pitch) $(arg gripper_mount_yaw)"/>
+      </xacro:dh_ag145_gripper>
+    </xacro:if>
+    <xacro:if value="${'$(arg gripper)' == 'ag95'}">
+      <xacro:include filename="$(find pxrd_cell)/urdf/dh_ag95_macro.xacro"/>
+      <xacro:dh_ag95_gripper parent="wrist3_link" prefix="">
+        <origin xyz="$(arg gripper_mount_x) $(arg gripper_mount_y) $(arg gripper_mount_z)"
+                rpy="$(arg gripper_mount_roll) $(arg gripper_mount_pitch) $(arg gripper_mount_yaw)"/>
+      </xacro:dh_ag95_gripper>
+    </xacro:if>
   </xacro:if>
 </robot>
